File: ESP1.kicad_sch (KiCad schematic)
At the start: 17 parts, among them U2 ESP32-S2-MINI-1-N4

Commit message: Last few files before production
Parts:
- BOOT1: value (none) -> SW_Push; footprint (none) -> Button_Switch_SMD:SW_SPST_Panasonic_EVQPL_3PL_5PL_PT_A08
- C1: value (none) -> 0.1uF; footprint (none) -> Capacitor_SMD:C_0603_1608Metric
- C2: value (none) -> 10uF; footprint (none) -> Capacitor_SMD:C_0805_2012Metric
- EN1: footprint (none) -> Button_Switch_SMD:SW_SPST_Panasonic_EVQPL_3PL_5PL_PT_A08
- J2: value (none) -> USB_C_Receptacle_USB2.0; footprint (none) -> USB-C-Power-tester:TYPE-C-31-M-12
- R2: value (none) -> 5.1K; footprint (none) -> Resistor_SMD:R_0603_1608Metric
- R4: value (none) -> 33R; footprint (none) -> Resistor_SMD:R_0603_1608Metric
- R6: value (none) -> 10K; footprint (none) -> Resistor_SMD:R_0603_1608Metric
- U2: value (none) -> ESP32-S2-MINI-1-N4; footprint (none) -> footprints:ESP32-S2-MINI-1-N4
Changed lines of the file:
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@@
       (effects (font (size 1.27 1.27)) hide)
     )
-    (property "Value" "" (id 1) (at 130.81 99.695 0))
+    (property "Value" "GND" (id 1) (at 130.81 99.695 0))
     (property "Footprint" "" (id 2) (at 130.81 95.25 0)
       (effects (font (size 1.27 1.27)) hide)
@@
     (property "Reference" "EN1" (id 0) (at 26.035 135.89 0))
     (property "Value" "SW_Push" (id 1) (at 26.035 138.43 0))
-    (property "Footprint" "" (id 2) (at 26.035 138.43 0)
+    (property "Footprint" "Button_Switch_SMD:SW_SPST_Panasonic_EVQPL_3PL_5PL_PT_A08" (id 2) (at 26.035 138.43 0)
       (effects (font (size 1.27 1.27)) hide)
     )
@@
       (effects (font (size 1.27 1.27)) hide)
     )
-    (property "Value" "" (id 1) (at 49.53 46.99 0))
+    (property "Value" "+3V3" (id 1) (at 49.53 46.99 0))
     (property "Footprint" "" (id 2) (at 49.53 52.07 0)
       (effects (font (size 1.27 1.27)) hide)
@@
       (effects (font (size 1.27 1.27)) hide)
     )
-    (property "Value" "" (id 1) (at 174.625 136.525 0))
+    (property "Value" "GND" (id 1) (at 174.625 136.525 0))
     (property "Footprint" "" (id 2) (at 174.625 131.445 0)
       (effects (font (size 1.27 1.27)) hide)
@@
       (effects (font (size 1.27 1.27)) (justify left))
     )
-    (property "Value" "" (id 1) (at 88.265 33.02 0)
-      (effects (font (size 1.27 1.27)) (justify left))
-    )
-    (property "Footprint" "" (id 2) (at 94.9452 34.29 0)
+    (property "Value" "0.1uF" (id 1) (at 88.265 33.02 0)
+      (effects (font (size 1.27 1.27)) (justify left))
+    )
+    (property "Footprint" "Capacitor_SMD:C_0603_1608Metric" (id 2) (at 94.9452 34.29 0)
       (effects (font (size 1.27 1.27)) hide)
     )
@@
       (effects (font (size 1.27 1.27)) hide)
     )
-    (property "Value" "" (id 1) (at 149.225 79.375 0))
+    (property "Value" "+5V" (id 1) (at 149.225 79.375 0))
     (property "Footprint" "" (id 2) (at 149.225 85.09 0)
       (effects (font (size 1.27 1.27)) hide)
@@
       (effects (font (size 1.27 1.27)) (justify right))
     )
-    (property "Value" "" (id 1) (at 178.435 100.9651 0)
+    (property "Value" "USB_C_Receptacle_USB2.0" (id 1) (at 178.435 100.9651 0)
       (effects (font (size 1.27 1.27)) (justify right))
     )
-    (property "Footprint" "" (id 2) (at 163.195 102.235 0)
+    (property "Footprint" "USB-C-Power-tester:TYPE-C-31-M-12" (id 2) (at 163.195 102.235 0)
       (effects (font (size 1.27 1.27)) hide)
     )
@@
     (in_bom yes) (on_board yes)
     (property "Reference" "R6" (id 0) (at 36.195 169.545 90))
-    (property "Value" "" (id 1) (at 38.1 169.545 90))
-    (property "Footprint" "" (id 2) (at 36.322 169.545 90)
+    (property "Value" "10K" (id 1) (at 38.1 169.545 90))
+    (property "Footprint" "Resistor_SMD:R_0603_1608Metric" (id 2) (at 36.322 169.545 90)
       (effects (font (size 1.27 1.27)) hide)
     )
@@
       (effects (font (size 1.27 1.27)) hide)
     )
-    (property "Value" "" (id 1) (at 220.345 137.16 0))
+    (property "Value" "PWR_FLAG" (id 1) (at 220.345 137.16 0))
     (property "Footprint" "" (id 2) (at 220.345 142.875 0)
       (effects (font (size 1.27 1.27)) hide)
@@
     (in_bom yes) (on_board yes) (fields_autoplaced)
     (property "Reference" "BOOT1" (id 0) (at 25.4 165.1 0))
-    (property "Value" "" (id 1) (at 25.4 167.64 0))
-    (property "Footprint" "" (id 2) (at 25.4 168.275 0)
+    (property "Value" "SW_Push" (id 1) (at 25.4 167.64 0))
+    (property "Footprint" "Button_Switch_SMD:SW_SPST_Panasonic_EVQPL_3PL_5PL_PT_A08" (id 2) (at 25.4 168.275 0)
       (effects (font (size 1.27 1.27)) hide)
     )
@@
       (effects (font (size 1.27 1.27)) (justify left))
     )
-    (property "Value" "" (id 1) (at 98.425 33.02 0)
-      (effects (font (size 1.27 1.27)) (justify left))
-    )
-    (property "Footprint" "" (id 2) (at 105.1052 34.29 0)
+    (property "Value" "10uF" (id 1) (at 98.425 33.02 0)
+      (effects (font (size 1.27 1.27)) (justify left))
+    )
+    (property "Footprint" "Capacitor_SMD:C_0805_2012Metric" (id 2) (at 105.1052 34.29 0)
       (effects (font (size 1.27 1.27)) hide)
     )
@@
       (effects (font (size 1.27 1.27)) hide)
     )
-    (property "Value" "" (id 1) (at 228.6 149.86 0))
+    (property "Value" "GND" (id 1) (at 228.6 149.86 0))
     (property "Footprint" "" (id 2) (at 228.6 144.78 0)
       (effects (font (size 1.27 1.27)) hide)
@@
     (in_bom yes) (on_board yes)
     (property "Reference" "R2" (id 0) (at 144.145 96.52 90))
-    (property "Value" "" (id 1) (at 144.145 94.615 90))
-    (property "Footprint" "" (id 2) (at 144.145 96.393 90)
+    (property "Value" "5.1K" (id 1) (at 144.145 94.615 90))
+    (property "Footprint" "Resistor_SMD:R_0603_1608Metric" (id 2) (at 144.145 96.393 90)
       (effects (font (size 1.27 1.27)) hide)
     )
@@
     (in_bom yes) (on_board yes)
     (property "Reference" "R4" (id 0) (at 144.145 106.68 90))
-    (property "Value" "" (id 1) (at 144.145 104.775 90))
-    (property "Footprint" "" (id 2) (at 144.145 102.997 90)
+    (property "Value" "33R" (id 1) (at 144.145 104.775 90))
+    (property "Footprint" "Resistor_SMD:R_0603_1608Metric" (id 2) (at 144.145 102.997 90)
       (effects (font (size 1.27 1.27)) hide)
     )
@@
       (effects (font (size 1.524 1.524)) (justify left))
     )
-    (property "Value" "" (id 1) (at 262.89 95.25 0)
+    (property "Value" "ESP32-S2-MINI-1-N4" (id 1) (at 262.89 95.25 0)
       (effects (font (size 1.524 1.524)) (justify left))
     )
-    (property "Footprint" "" (id 2) (at 248.92 42.164 0)
+    (property "Footprint" "footprints:ESP32-S2-MINI-1-N4" (id 2) (at 248.92 42.164 0)
       (effects (font (size 1.524 1.524)) hide)
     )
@@
     )
     (path "/11dc16dd-2246-40e3-849f-72301c294be5"
-      (reference "J1") (unit 1) (value "Conn_01x04_Male") (footprint "Connector_PinSocket_2.54mm:PinSocket_1x04_P2.54mm_Vertical")
+      (reference "J1") (unit 1) (value "Conn_01x04_Male") (footprint "Connector_PinHeader_2.54mm:PinHeader_1x04_P2.54mm_Vertical")
     )
     (path "/822d0909-74c7-4afe-acc0-b1ee5abf5d30"
